Commit message: [Gazebo sim] Simulation prepared with two robots in Noetic

File: robots/definition/sim/hokuyo.urdf.xacro (robot description, xacro)
@@ -2,4 +2,5 @@
 <robot name="sensor_hokuyo" xmlns:xacro="http://ros.org/wiki/xacro">
   <xacro:property name="M_PI" value="3.1415926535897931" />
+  <link name="base_link" />
   <xacro:macro name="hokuyo" params="name parent *origin ros_topic update_rate ray_count min_angle max_angle">
     <joint name="laser" type="fixed">

File: robots/definition/sim/kobuki_hexagons_asus_xtion_pro.urdf.xacro (robot description, xacro)
@@ -6,5 +6,5 @@
 -->
 <robot name="turtlebot" xmlns:xacro="http://ros.org/wiki/xacro">
-	<xacro:include filename="$(find robots)/definition/sim/urdf/common_properties.urdf.xacro"/>
+  <xacro:include filename="$(find robots)/definition/sim/urdf/common_properties.urdf.xacro"/>
   <xacro:include filename="$(find robots)/definition/sim/urdf/turtlebot_properties.urdf.xacro"/>
   <!-- Bases -->
@@ -22,5 +22,5 @@
   <sensor_asus_xtion_pro          parent="base_link"/>
 <!--  <sensor_hokuyo 		              parent="base_link" name="laser0" ros_topic="scan" update_rate="40" ray_count="1081" min_angle="135" max_angle="-135" />-->
-  <include filename="$(find robots)/definition/sim/hokuyo.urdf.xacro" />
+  <xacro:include filename="$(find robots)/definition/sim/hokuyo.urdf.xacro" />
   <xacro:hokuyo name="laser0" parent="base_link" ros_topic="scan" update_rate="40" ray_count="1081" min_angle="135" max_angle="-135">
       <origin xyz="0.0 0.0 0.08" rpy="${M_PI} 0 0"/>
